File: vacuum_pickup_tool/vacuum_pickup_tool.sch (KiCad schematic (older format))
At the start: 19 parts, among them J1 Barrel_Jack, J2 AudioJack3, J3 JST_PH_01x02_Male, J4 JST_PH_01x02_Male, U1 Amazon_Small_Buck, U2 NCE6005AS

Commit message: Make v1.0
Parts:
- U2: MPN (none) -> NCE6005AS
Changed lines of the file:
@@
 EESchema Schematic File Version 4
-LIBS:vacuum_pickup_tool-cache
 EELAYER 30 0
 EELAYER END
@@
 F 2 "lib_fp:SOP-8_3.76x4.96mm_P1.27mm" H 7100 2200 50  0001 C CNN
 F 3 "" H 7100 2200 50  0001 C CNN
+F 4 "NCE6005AS" H 6950 2200 50  0001 C CNN "MPN"
 	2    6950 2200
 	1    0    0    -1
@@
 F 1 "Barrel_Jack" H 1407 4234 50  0000 C CNN
 F 2 "lib_fp:SOFNG_DC005-T20" H 1400 3960 50  0001 C CNN
-F 3 "https://datasheet.lcsc.com/szlcsc/SOFNG-DC-050-T20_C114916.pdf" H 1400 3960 50  0001 C CNN
+F 3 "https://datasheet.lcsc.com/szlcsc/1908270930_Boom-Precision-Elec-DC-005-5-5-2-0MM_C16214.pdf" H 1400 3960 50  0001 C CNN
 F 4 "DC005-T20" H 1350 4000 50  0001 C CNN "MPN"
 	1    1350 4000
