File: vacuum_pickup_tool/vacuum_pickup_tool.kicad_pcb (KiCad board)
At the start: 2 copper layers, 58.4 x 58.4 mm, 19 parts, among them J1 Barrel_Jack, J2 AudioJack3, J3 JST_PH_01x02_Male, J4 JST_PH_01x02_Male, U1 Amazon_Small_Buck, U2 NCE6005AS

Commit message: Make v1.0
Parts:
- added G***: LOGO, lib_fp:bird_with_pants_small_flipped, F.Cu at (0.00, 44.5)
Changed lines of the file:
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@@
-(kicad_pcb (version 20171130) (host pcbnew "(5.1.4)-1")
+(kicad_pcb (version 20171130) (host pcbnew "(5.1.4-0)")
   (general
     (thickness 1.6)
@@
     (tracks 101)
     (zones 0)
-    (modules 19)
+    (modules 20)
     (nets 12)
   )
@@
   )
   (setup
-    (last_trace_width 0.4)
+    (last_trace_width 0.25)
     (user_trace_width 0.2)
     (user_trace_width 0.4)
@@
       (outputformat 1)
       (mirror false)
-      (drillshape 1)
+      (drillshape 0)
       (scaleselection 1)
-      (outputdirectory ""))
+      (outputdirectory "plots/"))
   )
   (net 0 "")
@@
     (uvia_drill 0.1)
   )
+  (module lib_fp:bird_with_pants_small_flipped (layer F.Cu)
+    (at 0 44.45 90)
+    (fp_text reference G*** (at 0 0 90) (layer F.SilkS) hide
+      (effects (font (size 1.524 1.524) (thickness 0.3)))
+    )
+    (fp_text value LOGO (at 0.75 0 90) (layer F.SilkS) hide
+      (effects (font (size 1.524 1.524) (thickness 0.3)))
+    )
+    (fp_poly (pts (xy 0.4953 0.8255) (xy -1.3208 0.8255) (xy -1.6002 1.5875) (xy 0.381 1.5875)) (layer F.SilkS) (width 0.1))
+    (fp_poly (pts (xy 1.143 -1.524) (xy -0.4445 -1.524) (xy -1.2192 0.5715) (xy 0.5334 0.5715)
+      (xy 0.7874 -1.143)) (layer F.SilkS) (width 0.1))
+  )
   (module Diode_SMD:D_SMA (layer F.Cu)
     (at 35.814 38.1 270)
@@
     (fp_line (start 0 -4.5) (end 13.5 -4.5) (layer F.SilkS) (width 0.15))
     (fp_line (start 0 -4.5) (end 0 4.5) (layer F.SilkS) (width 0.15))
-    (pad 3 thru_hole rect (at 13.5 0 180) (size 2 4) (drill oval 0.8 3.5) (layers *.Cu *.Mask))
+    (pad 1 thru_hole rect (at 13.5 0 180) (size 2 4) (drill oval 0.8 3.5) (layers *.Cu *.Mask)
+      (net 6 +12V))
     (pad 2 thru_hole rect (at 7.5 0 180) (size 2 4) (drill oval 0.8 3) (layers *.Cu *.Mask)
       (net 1 GND))
-    (pad 1 thru_hole rect (at 11 4.8 180) (size 4 2) (drill oval 3 0.8) (layers *.Cu *.Mask)
-      (net 6 +12V))
+    (pad 2 thru_hole rect (at 11 4.8 180) (size 4 2) (drill oval 3 0.8) (layers *.Cu *.Mask)
+      (net 1 GND))
     (model "${KIPRJMOD}/lib_3d/DC Jack v2.step"
       (offset (xyz 7.5 0 0))
@@
     (effects (font (size 1 1) (thickness 0.15)))
   )
-  (gr_text "Vacuum Pickup Tool Control Board v1.0\npantsforbirds.com" (at 0 45.085 90) (layer F.SilkS)
+  (gr_text "Vacuum Pickup Tool Control Board v1.0\npantsforbirds.com" (at 0 40.64 90) (layer F.SilkS)
     (effects (font (size 1 1) (thickness 0.15)) (justify left))
   )
@@
   (segment (start 42.545 42.545) (end 42.545 38.1) (width 0.4) (layer F.Cu) (net 2))
   (via (at 42.545 38.1) (size 0.8) (drill 0.4) (layers F.Cu B.Cu) (net 2))
+  (segment (start 45.085 45.72) (end 45.085 47.0875) (width 0.4) (layer F.Cu) (net 2) (status 10))
+  (segment (start 42.545 42.545) (end 42.545 43.18) (width 0.4) (layer F.Cu) (net 2))
+  (segment (start 42.545 43.18) (end 45.085 45.72) (width 0.4) (layer F.Cu) (net 2) (status 20))
+  (segment (start 45.085 47.0875) (end 45.085 47.625) (width 0.4) (layer F.Cu) (net 2) (status 20))
+  (segment (start 45.085 45.72) (end 49.53 45.72) (width 0.4) (layer F.Cu) (net 2) (status 30))
   (segment (start 4.514999 30.549999) (end 4.514999 8.820001) (width 0.4) (layer F.Cu) (net 3))
   (segment (start 5.715 31.75) (end 4.514999 30.549999) (width 0.4) (layer F.Cu) (net 3) (status 10))
@@
   (segment (start 38.1 33.02) (end 38.1 38.1) (width 1) (layer B.Cu) (net 7))
   (segment (start 38.1 38.1) (end 38.1 39.37) (width 1) (layer F.Cu) (net 7))
+  (segment (start 35.5575 28.575) (end 35.5575 29.8425) (width 1) (layer F.Cu) (net 7) (status 30))
   (segment (start 25.7555 5.08) (end 12.065 5.08) (width 0.4) (layer F.Cu) (net 8) (status 30))
   (segment (start 12.065 2.54) (end 25.4 2.54) (width 0.4) (layer F.Cu) (net 9) (status 30))
@@
   (via (at 39.37 48.26) (size 0.8) (drill 0.4) (layers F.Cu B.Cu) (net 10))
   (segment (start 39.37 43.18) (end 39.37 48.26) (width 1) (layer B.Cu) (net 10))
-  (segment (start 45.085 45.72) (end 45.085 47.0875) (width 0.4) (layer F.Cu) (net 2) (status 10))
-  (segment (start 42.545 42.545) (end 42.545 43.18) (width 0.4) (layer F.Cu) (net 2))
-  (segment (start 42.545 43.18) (end 45.085 45.72) (width 0.4) (layer F.Cu) (net 2) (status 20))
-  (segment (start 45.085 47.0875) (end 45.085 47.625) (width 0.4) (layer F.Cu) (net 2) (status 20))
-  (segment (start 45.085 45.72) (end 49.53 45.72) (width 0.4) (layer F.Cu) (net 2) (status 30))
-  (segment (start 35.5575 28.575) (end 35.5575 29.8425) (width 1) (layer F.Cu) (net 7) (status 30))
   (segment (start 35.5575 26.035) (end 35.5575 27.3025) (width 1) (layer F.Cu) (net 10) (status 30))
   (via (at 42.545 52.07) (size 0.8) (drill 0.4) (layers F.Cu B.Cu) (net 11))

Commit message: Add hella files and README parts
Parts:
- added J5: JST_PH_01x02_Male, Connector_JST:JST_PH_B2B-PH-K_1x02_P2.00mm_Vertical, F.Cu at (29.5, 33.8)
- moved J3 2.74 mm to (29.5, 39.4), turned to 0 degrees
Connections:
- J2 pad S: GND -> (no net)
Routing:
- net Net-(D1-Pad2): track 20.3 -> 24.9 mm
- net GND: track 35.0 -> 32.9 mm, vias 11 -> 9
Other:
- board text added: "Vacuum Pickup Tool Control Board v1.1 pantsforbirds.com"
- board text removed: "Vacuum Pickup Tool Control Board v1.0 pantsforbirds.com"
Changed lines of the file:
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@@
-(kicad_pcb (version 20171130) (host pcbnew "(5.1.4-0)")
+(kicad_pcb (version 20171130) (host pcbnew "(5.1.4)-1")
   (general
     (thickness 1.6)
     (drawings 10)
-    (tracks 101)
+    (tracks 99)
     (zones 0)
-    (modules 20)
+    (modules 21)
     (nets 12)
   )
@@
   )
   (setup
-    (last_trace_width 0.25)
+    (last_trace_width 1)
     (user_trace_width 0.2)
     (user_trace_width 0.4)
@@
     (fp_line (start 5.842 3) (end 7 3) (layer F.SilkS) (width 0.15))
     (fp_line (start -4 -3) (end -0.889 -3) (layer F.SilkS) (width 0.15))
-    (pad S smd rect (at -2 5.5 180) (size 1.5 3.5) (drill (offset 0 -1.75)) (layers F.Cu F.Paste F.Mask)
-      (net 1 GND))
+    (pad S smd rect (at -2 5.5 180) (size 1.5 3.5) (drill (offset 0 -1.75)) (layers F.Cu F.Paste F.Mask))
     (pad R smd rect (at 0 -5.5 180) (size 1.5 3.5) (drill (offset 0 1.75)) (layers F.Cu F.Paste F.Mask)
       (net 2 /TRIGGER_SWITCH))
@@
   )
   (module Connector_JST:JST_PH_B2B-PH-K_1x02_P2.00mm_Vertical (layer F.Cu)
-    (at 30.48 36.83 270)
+    (at 29.464 39.37)
     (descr "JST PH series connector, B2B-PH-K (http://www.jst-mfg.com/product/pdf/eng/ePH.pdf), generated with kicad-footprint-generator")
     (tags "connector JST PH side entry")
-    (fp_text reference J3 (at 1 -2.9 90) (layer F.SilkS)
-      (effects (font (size 1 1) (thickness 0.15)))
-    )
-    (fp_text value JST_PH_01x02_Male (at 1 4 90) (layer F.Fab)
-      (effects (font (size 1 1) (thickness 0.15)))
-    )
-    (fp_text user %R (at 1 1.5 90) (layer F.Fab)
+    (fp_text reference J3 (at 1 -2.9) (layer F.SilkS)
+      (effects (font (size 1 1) (thickness 0.15)))
+    )
+    (fp_text value JST_PH_01x02_Male (at 1 4) (layer F.Fab)
+      (effects (font (size 1 1) (thickness 0.15)))
+    )
+    (fp_text user %R (at 1 1.5) (layer F.Fab)
       (effects (font (size 1 1) (thickness 0.15)))
     )
@@
     (fp_line (start -2.06 2.91) (end 4.06 2.91) (layer F.SilkS) (width 0.12))
     (fp_line (start -2.06 -1.81) (end -2.06 2.91) (layer F.SilkS) (width 0.12))
-    (pad 2 thru_hole oval (at 2 0 270) (size 1.2 1.75) (drill 0.75) (layers *.Cu *.Mask)
+    (pad 2 thru_hole oval (at 2 0) (size 1.2 1.75) (drill 0.75) (layers *.Cu *.Mask)
       (net 7 "Net-(D1-Pad2)"))
-    (pad 1 thru_hole roundrect (at 0 0 270) (size 1.2 1.75) (drill 0.75) (layers *.Cu *.Mask) (roundrect_rratio 0.208333)
+    (pad 1 thru_hole roundrect (at 0 0) (size 1.2 1.75) (drill 0.75) (layers *.Cu *.Mask) (roundrect_rratio 0.208333)
       (net 6 +12V))
     (model ${KISYS3DMOD}/Connector_JST.3dshapes/JST_PH_B2B-PH-K_1x02_P2.00mm_Vertical.wrl
@@
     )
   )
+  (module Connector_JST:JST_PH_B2B-PH-K_1x02_P2.00mm_Vertical (layer F.Cu)
+    (at 29.464 33.782)
+    (descr "JST PH series connector, B2B-PH-K (http://www.jst-mfg.com/product/pdf/eng/ePH.pdf), generated with kicad-footprint-generator")
+    (tags "connector JST PH side entry")
+    (fp_text reference J5 (at 1 -2.9) (layer F.SilkS)
+      (effects (font (size 1 1) (thickness 0.15)))
+    )
+    (fp_text value JST_PH_01x02_Male (at 1 4) (layer F.Fab)
+      (effects (font (size 1 1) (thickness 0.15)))
+    )
+    (fp_line (start -2.06 -1.81) (end -2.06 2.91) (layer F.SilkS) (width 0.12))
+    (fp_line (start -2.06 2.91) (end 4.06 2.91) (layer F.SilkS) (width 0.12))
+    (fp_line (start 4.06 2.91) (end 4.06 -1.81) (layer F.SilkS) (width 0.12))
+    (fp_line (start 4.06 -1.81) (end -2.06 -1.81) (layer F.SilkS) (width 0.12))
+    (fp_line (start -0.3 -1.81) (end -0.3 -2.01) (layer F.SilkS) (width 0.12))
+    (fp_line (start -0.3 -2.01) (end -0.6 -2.01) (layer F.SilkS) (width 0.12))
+    (fp_line (start -0.6 -2.01) (end -0.6 -1.81) (layer F.SilkS) (width 0.12))
+    (fp_line (start -0.3 -1.91) (end -0.6 -1.91) (layer F.SilkS) (width 0.12))
+    (fp_line (start 0.5 -1.81) (end 0.5 -1.2) (layer F.SilkS) (width 0.12))
+    (fp_line (start 0.5 -1.2) (end -1.45 -1.2) (layer F.SilkS) (width 0.12))
+    (fp_line (start -1.45 -1.2) (end -1.45 2.3) (layer F.SilkS) (width 0.12))
+    (fp_line (start -1.45 2.3) (end 3.45 2.3) (layer F.SilkS) (width 0.12))
+    (fp_line (start 3.45 2.3) (end 3.45 -1.2) (layer F.SilkS) (width 0.12))
+    (fp_line (start 3.45 -1.2) (end 1.5 -1.2) (layer F.SilkS) (width 0.12))
+    (fp_line (start 1.5 -1.2) (end 1.5 -1.81) (layer F.SilkS) (width 0.12))
+    (fp_line (start -2.06 -0.5) (end -1.45 -0.5) (layer F.SilkS) (width 0.12))
+    (fp_line (start -2.06 0.8) (end -1.45 0.8) (layer F.SilkS) (width 0.12))
+    (fp_line (start 4.06 -0.5) (end 3.45 -0.5) (layer F.SilkS) (width 0.12))
+    (fp_line (start 4.06 0.8) (end 3.45 0.8) (layer F.SilkS) (width 0.12))
+    (fp_line (start 0.9 2.3) (end 0.9 1.8) (layer F.SilkS) (width 0.12))
+    (fp_line (start 0.9 1.8) (end 1.1 1.8) (layer F.SilkS) (width 0.12))
+    (fp_line (start 1.1 1.8) (end 1.1 2.3) (layer F.SilkS) (width 0.12))
+    (fp_line (start 1 2.3) (end 1 1.8) (layer F.SilkS) (width 0.12))
+    (fp_line (start -1.11 -2.11) (end -2.36 -2.11) (layer F.SilkS) (width 0.12))
+    (fp_line (start -2.36 -2.11) (end -2.36 -0.86) (layer F.SilkS) (width 0.12))
+    (fp_line (start -1.11 -2.11) (end -2.36 -2.11) (layer F.Fab) (width 0.1))
+    (fp_line (start -2.36 -2.11) (end -2.36 -0.86) (layer F.Fab) (width 0.1))
+    (fp_line (start -1.95 -1.7) (end -1.95 2.8) (layer F.Fab) (width 0.1))
+    (fp_line (start -1.95 2.8) (end 3.95 2.8) (layer F.Fab) (width 0.1))
+    (fp_line (start 3.95 2.8) (end 3.95 -1.7) (layer F.Fab) (width 0.1))
+    (fp_line (start 3.95 -1.7) (end -1.95 -1.7) (layer F.Fab) (width 0.1))
+    (fp_line (start -2.45 -2.2) (end -2.45 3.3) (layer F.CrtYd) (width 0.05))
+    (fp_line (start -2.45 3.3) (end 4.45 3.3) (layer F.CrtYd) (width 0.05))
+    (fp_line (start 4.45 3.3) (end 4.45 -2.2) (layer F.CrtYd) (width 0.05))
+    (fp_line (start 4.45 -2.2) (end -2.45 -2.2) (layer F.CrtYd) (width 0.05))
+    (fp_text user %R (at 1 1.5) (layer F.Fab)
+      (effects (font (size 1 1) (thickness 0.15)))
+    )
+    (pad 1 thru_hole roundrect (at 0 0) (size 1.2 1.75) (drill 0.75) (layers *.Cu *.Mask) (roundrect_rratio 0.208333)
+      (net 6 +12V))
+    (pad 2 thru_hole oval (at 2 0) (size 1.2 1.75) (drill 0.75) (layers *.Cu *.Mask)
+      (net 7 "Net-(D1-Pad2)"))
+    (model ${KISYS3DMOD}/Connector_JST.3dshapes/JST_PH_B2B-PH-K_1x02_P2.00mm_Vertical.wrl
+      (at (xyz 0 0 0))
+      (scale (xyz 1 1 1))
+      (rotate (xyz 0 0 0))
+    )
+  )
   (gr_text "Adjust output to +5V\nbefore installation!" (at 41.275 15.24) (layer F.SilkS)
     (effects (font (size 1 1) (thickness 0.15)))
   )
-  (gr_text "Vacuum Pickup Tool Control Board v1.0\npantsforbirds.com" (at 0 40.64 90) (layer F.SilkS)
+  (gr_text "Vacuum Pickup Tool Control Board v1.1\npantsforbirds.com" (at 0 40.64 90) (layer F.SilkS)
     (effects (font (size 1 1) (thickness 0.15)) (justify left))
   )
@@
   (segment (start 44.435 35.14) (end 44.435 34.305) (width 1) (layer F.Cu) (net 1) (status 10))
   (segment (start 44.435 33.035) (end 44.45 33.02) (width 1) (layer F.Cu) (net 1))
-  (via (at 51.435 33.02) (size 0.8) (drill 0.4) (layers F.Cu B.Cu) (net 1))
-  (segment (start 51.435 35.14) (end 51.435 34.29) (width 1) (layer F.Cu) (net 1) (status 10))
-  (segment (start 51.435 34.29) (end 51.435 33.02) (width 1) (layer F.Cu) (net 1))
-  (via (at 51.435 34.29) (size 0.8) (drill 0.4) (layers F.Cu B.Cu) (net 1))
   (segment (start 44.435 34.305) (end 44.435 33.035) (width 1) (layer F.Cu) (net 1))
   (via (at 44.435 34.305) (size 0.8) (drill 0.4) (layers F.Cu B.Cu) (net 1))
@@
   (segment (start 26.67 29.845) (end 27.305 29.845) (width 0.4) (layer F.Cu) (net 5))
   (segment (start 35.5575 29.8425) (end 38.1 32.385) (width 1) (layer F.Cu) (net 7) (status 10))
-  (segment (start 38.1 39.37) (end 37.465 40.005) (width 1) (layer F.Cu) (net 7))
-  (segment (start 37.465 40.005) (end 31.75 40.005) (width 1) (layer F.Cu) (net 7))
-  (segment (start 31.75 40.005) (end 30.48 38.735) (width 1) (layer F.Cu) (net 7) (status 20))
+  (segment (start 38.1 33.02) (end 38.1 38.1) (width 1) (layer B.Cu) (net 7))
+  (via (at 38.1 38.1) (size 0.8) (drill 0.4) (layers F.Cu B.Cu) (net 7))
+  (segment (start 38.1 32.385) (end 38.1 33.02) (width 1) (layer F.Cu) (net 7))
   (via (at 38.1 33.02) (size 0.8) (drill 0.4) (layers F.Cu B.Cu) (net 7))
-  (segment (start 38.1 32.385) (end 38.1 33.02) (width 1) (layer F.Cu) (net 7))
-  (via (at 38.1 38.1) (size 0.8) (drill 0.4) (layers F.Cu B.Cu) (net 7))
-  (segment (start 38.1 33.02) (end 38.1 38.1) (width 1) (layer B.Cu) (net 7))
-  (segment (start 38.1 38.1) (end 38.1 39.37) (width 1) (layer F.Cu) (net 7))
   (segment (start 35.5575 28.575) (end 35.5575 29.8425) (width 1) (layer F.Cu) (net 7) (status 30))
+  (segment (start 31.464 33.782) (end 31.464 39.37) (width 1) (layer F.Cu) (net 7))
+  (segment (start 32.194 40.1) (end 31.464 39.37) (width 1) (layer F.Cu) (net 7))
+  (segment (start 35.814 40.1) (end 32.194 40.1) (width 1) (layer F.Cu) (net 7))
+  (segment (start 37.714 40.1) (end 35.814 40.1) (width 1) (layer F.Cu) (net 7))
+  (segment (start 38.1 39.714) (end 37.714 40.1) (width 1) (layer F.Cu) (net 7))
+  (segment (start 38.1 38.1) (end 38.1 39.714) (width 1) (layer F.Cu) (net 7))
   (segment (start 25.7555 5.08) (end 12.065 5.08) (width 0.4) (layer F.Cu) (net 8) (status 30))
   (segment (start 12.065 2.54) (end 25.4 2.54) (width 0.4) (layer F.Cu) (net 9) (status 30))
@@
   (segment (start 35.5575 26.035) (end 35.5575 27.3025) (width 1) (layer F.Cu) (net 10) (status 30))
   (via (at 42.545 52.07) (size 0.8) (drill 0.4) (layers F.Cu B.Cu) (net 11))
-  (segment (start 43.51 45.72) (end 43.51 51.105) (width 0.4) (layer F.Cu) (net 11))
+  (segment (start 43.51 45.72) (end 43.51 51.105) (width 0.4) (layer F.Cu) (net 11) (status 10))
   (segment (start 43.51 51.105) (end 42.545 52.07) (width 0.4) (layer F.Cu) (net 11))
   (via (at 37.465 52.07) (size 0.8) (drill 0.4) (layers F.Cu B.Cu) (net 11))
